Commit message: Insert  Ultrassonic :dart:

File: src/my_bot/description/robot_core.xacro (robot description, xacro)
@@ -125,4 +125,7 @@
             <material name="black"/>
         </collision>
+        <xacro:inertial_sphere mass="0.3" radius="0.05">
+            <origin xyz="0 0 0" rpy="0 0 0"/>
+        </xacro:inertial_sphere>
     </link>
     <gazebo reference="caster_wheel">

File: src/my_bot/description/sensor.xacro (robot description, xacro)
@@ -1,10 +1,11 @@
 <?xml version="1.0"?>
 <robot xmlns:xacro="http://www.ros.org/wiki/xacro" >
-    <joint name="laser_joint" type="fixed">
+    <!-- ====================== Direita Sensor ultrassonico ====================-->
+    <joint name="laser_joint1" type="fixed">
         <parent link="chassis"/>
-        <child link="laser_frame"/>
-        <origin xyz="0.250 0.100 0.175" rpy="0 0 0.3"/>
+        <child link="laser_frame1"/>
+        <origin xyz="0.250 0.100 0.160" rpy="0 0 0.3"/>
     </joint>
-    <link name="laser_frame">
+    <link name="laser_frame1">
         <visual>
             <geometry>
@@ -15,15 +16,15 @@
         <collision>
             <geometry>
-                <cylinder radius="0.05" length="0.04"/>
+                <box size="0.03 0.03 0.015"/>
             </geometry>
         </collision>
-        <xacro:inertial_cylinder mass="0.1" length="0.04" radius="0.05">
-            <origin xyz="0 0 0" rpy="0 0 0"/>
-        </xacro:inertial_cylinder>
+        <xacro:inertial_box mass="0.02" x="0.03" y="0.03" z="0.015">
+            <origin xyz="0.250 0.100 0.160" rpy="0 0 0.3"/>
+        </xacro:inertial_box>
     </link>
-    <gazebo reference="laser_frame">
+    <gazebo reference="laser_frame1">
         <material>Gazebo/Red</material>
         <pose>0 0 0 0 0 0</pose>
-        <sensor name="laser" type="ray">
+        <sensor name="laser1" type="ray">
             <always_on>true</always_on>
             <visualize>true</visualize>
@@ -55,10 +56,138 @@
                 </noise>
             </ray>
-            <plugin name="laser_controller" filename="libgazebo_ros_ray_sensor.so">
+            <plugin name="laser_controller1" filename="libgazebo_ros_ray_sensor.so">
                 <ros>
                     <argument>~/out:=scan</argument>
                 </ros>
                 <output_type>sensor_msgs/LaserScan</output_type>
-                <frame_name>laser_frame</frame_name>
+                <frame_name>laser_frame1</frame_name>
+            </plugin>
+        </sensor>
+   </gazebo>
+   <!-- ====================== Esquerda Sensor ultrassonico ====================-->
+    <joint name="laser_joint2" type="fixed">
+        <parent link="chassis"/>
+        <child link="laser_frame2"/>
+        <origin xyz="0.250 -0.100 0.160" rpy="0 0 -0.3"/>
+    </joint>
+    <link name="laser_frame2">
+        <visual>
+            <geometry>
+                <box size="0.03 0.03 0.015"/>
+            </geometry>
+            <material name="red"/>
+        </visual>
+        <collision>
+            <geometry>
+                <box size="0.03 0.03 0.015"/>
+            </geometry>
+        </collision>
+        <xacro:inertial_box mass="0.02" x="0.03" y="0.03" z="0.015">
+            <origin xyz="0.250 -0.100 0.160" rpy="0 0 -0.3"/>
+        </xacro:inertial_box>
+    </link>
+    <gazebo reference="laser_frame2">
+        <material>Gazebo/Red</material>
+        <pose>0 0 0 0 0 0</pose>
+        <sensor name="laser2" type="ray">
+            <always_on>true</always_on>
+            <visualize>true</visualize>
+            <update_rate>10</update_rate>
+            <ray>
+                <scan>
+                    <horizontal>
+                        <samples>10</samples>
+                        <resolution>1.000000</resolution>
+                        <min_angle>-0.12</min_angle>
+                        <max_angle>0.12</max_angle>
+                    </horizontal>
+                    <vertical>
+                        <samples>10</samples>
+                        <resolution>1.000000</resolution>
+                         <min_angle>-0.08</min_angle>
+                         <max_angle>0.09</max_angle>
+                    </vertical>
+                </scan>
+                <range>
+                    <min>0.1</min>
+                    <max>2.3</max>
+                    <resolution>0.01</resolution>
+                </range>
+                <noise>
+                    <type>gaussian</type>
+                    <mean>0.0</mean>
+                    <stddev>0.01</stddev>
+                </noise>
+            </ray>
+            <plugin name="laser_controller2" filename="libgazebo_ros_ray_sensor.so">
+                <ros>
+                    <argument>~/out:=scan</argument>
+                </ros>
+                <output_type>sensor_msgs/LaserScan</output_type>
+                <frame_name>laser_frame2</frame_name>
+            </plugin>
+        </sensor>
+   </gazebo>
+   <!-- ====================== Centro Sensor ultrassonico ====================-->
+    <joint name="laser_joint3" type="fixed">
+        <parent link="chassis"/>
+        <child link="laser_frame3"/>
+        <origin xyz="0.250 0 0.160" rpy="0 0 0"/>
+    </joint>
+    <link name="laser_frame3">
+        <visual>
+            <geometry>
+                <box size="0.03 0.03 0.015"/>
+            </geometry>
+            <material name="red"/>
+        </visual>
+        <collision>
+            <geometry>
+                <box size="0.03 0.03 0.015"/>
+            </geometry>
+        </collision>
+        <xacro:inertial_box mass="0.02" x="0.03" y="0.03" z="0.015">
+            <origin xyz="0.250 0 0.160" rpy="0 0 0"/>
+        </xacro:inertial_box>
+    </link>
+    <gazebo reference="laser_frame3">
+        <material>Gazebo/Red</material>
+        <pose>0 0 0 0 0 0</pose>
+        <sensor name="laser3" type="ray">
+            <always_on>true</always_on>
+            <visualize>true</visualize>
+            <update_rate>10</update_rate>
+            <ray>
+                <scan>
+                    <horizontal>
+                        <samples>10</samples>
+                        <resolution>1.000000</resolution>
+                        <min_angle>-0.12</min_angle>
+                        <max_angle>0.12</max_angle>
+                    </horizontal>
+                    <vertical>
+                        <samples>10</samples>
+                        <resolution>1.000000</resolution>
+                         <min_angle>-0.08</min_angle>
+                         <max_angle>0.09</max_angle>
+                    </vertical>
+                </scan>
+                <range>
+                    <min>0.1</min>
+                    <max>2.3</max>
+                    <resolution>0.01</resolution>
+                </range>
+                <noise>
+                    <type>gaussian</type>
+                    <mean>0.0</mean>
+                    <stddev>0.01</stddev>
+                </noise>
+            </ray>
+            <plugin name="laser_controller3" filename="libgazebo_ros_ray_sensor.so">
+                <ros>
+                    <argument>~/out:=scan</argument>
+                </ros>
+                <output_type>sensor_msgs/LaserScan</output_type>
+                <frame_name>laser_frame3</frame_name>
             </plugin>
         </sensor>
